File: macro-kb.kicad_pcb (KiCad board)
At the start: 2 copper layers, 68.3 x 49.2 mm, 52 parts, among them SW1 SW_Push, U1 ATmega32U2-MU, Y1 16MHz 18pF

Commit message: routed
Routing:
- added copper zone on B.Cu, net GND
- added copper zone on F.Cu, net GND
Other:
- board text added: "JM 2019"
- board text added: "eletrcISTas"
- board text added: "macroKB version 1.0"

Commit message: final version (hopefully)
Parts:
- added R5: 470, Resistor_SMD:R_0603_1608Metric, B.Cu at (113.9, 83.9)
- D1, D2, D3, D4, D5, D6: value SOD-123 -> SOD-123F; footprint Diode_SMD:D_SOD-123 -> Diode_SMD:D_SOD-123F
- F1: value Polyfuse -> 500mA
Connections:
- net ROW2 renamed Net-(U1-Pad19)
- D11 pad 3: KEY_LEDS -> Net-(D11-Pad3)
- D16 pad 1: Net-(D16-Pad1) -> UNDERGLOW_LEDS
- U1 pad 9: UNDERGLOW_LEDS -> Net-(U1-Pad9)
Routing:
- net UNDERGLOW_LEDS: track 102.3 -> 8.57 mm, vias 6 -> 1
- net KEY_LEDS: track 75.9 -> 70.7 mm, vias 5 -> 4
- net Net-(D11-Pad3): track 0.00 -> 3.60 mm, vias 0 -> 1
